File: BIFROST-3S.kicad_pcb (KiCad board)
At the start: 2 copper layers, 46 x 23 mm, 14 parts, among them J1 B6B-XH-A_LF__SN_, J2 Conn_01x12, J3 B4B-XH-A_LF__SN_, J4 XT30PW-M

Commit message: Layout 6.0
Routing:
- added copper zone on B.Cu, net /+BATT
- added copper zone on B.Cu, net /PACK+_RAW
- added copper zone on In1.Cu, net GND
- added copper zone on In2.Cu, net GND
Other:
- copper layers 2 -> 4
Changed lines of the file:
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@@
 	(layers
 		(0 "F.Cu" signal)
+		(4 "In1.Cu" signal)
+		(6 "In2.Cu" signal)
 		(2 "B.Cu" signal)
 		(9 "F.Adhes" user "F.Adhesive")
@@
 			)
 			(layer "dielectric 1"
+				(type "prepreg")
+				(thickness 0.1)
+				(material "FR4")
+				(epsilon_r 4.5)
+				(loss_tangent 0.02)
+			)
+			(layer "In1.Cu"
+				(type "copper")
+				(thickness 0.035)
+			)
+			(layer "dielectric 2"
 				(type "core")
-				(thickness 1.51)
+				(thickness 1.24)
+				(material "FR4")
+				(epsilon_r 4.5)
+				(loss_tangent 0.02)
+			)
+			(layer "In2.Cu"
+				(type "copper")
+				(thickness 0.035)
+			)
+			(layer "dielectric 3"
+				(type "prepreg")
+				(thickness 0.1)
 				(material "FR4")
 				(epsilon_r 4.5)
@@
 		(layer "B.Cu")
 		(hatch edge 0.5)
+		(priority 3)
+		(connect_pads yes
+			(clearance 0.5)
+		)
+		(min_thickness 0.25)
+		(filled_areas_thickness no)
+		(fill yes
+			(thermal_gap 0.5)
+			(thermal_bridge_width 0.5)
+		)
+		(polygon
+			(pts
+				(xy 123.39 120.28) (xy 123.83 120.72) (xy 156.76 120.72) (xy 157.1 120.38) (xy 157.1 119.86) (xy 146.94 109.7)
+				(xy 146.94 99.1) (xy 146.65 98.81) (xy 123.79 98.81) (xy 123.39 99.21)
+			)
+		)
+	)
+	(zone
+		(net 6)
+		(net_name "/PACK+_RAW")
+		(layer "B.Cu")
+		(hatch edge 0.5)
+		(connect_pads yes
+			(clearance 0.5)
+		)
+		(min_thickness 0.25)
+		(filled_areas_thickness no)
+		(fill yes
+			(thermal_gap 0.5)
+			(thermal_bridge_width 0.5)
+		)
+		(polygon
+			(pts
+				(xy 147.83 103.69) (xy 167.91 103.69) (xy 168.23 103.37) (xy 168.23 99.03) (xy 167.97 98.77) (xy 147.77 98.77)
+				(xy 147.51 99.03) (xy 147.51 103.37)
+			)
+		)
+	)
+	(zone
+		(net 3)
+		(net_name "/+BATT")
+		(layer "B.Cu")
+		(hatch edge 0.5)
+		(priority 2)
+		(connect_pads yes
+			(clearance 0.5)
+		)
+		(min_thickness 0.25)
+		(filled_areas_thickness no)
+		(fill yes
+			(thermal_gap 0.5)
+			(thermal_bridge_width 0.5)
+		)
+		(polygon
+			(pts
+				(xy 148.02 104.46) (xy 167.75 104.46) (xy 168.19 104.9) (xy 168.19 120.23) (xy 167.68 120.74) (xy 158.6 120.74)
+				(xy 147.66 109.8) (xy 147.66 104.82)
+			)
+		)
+	)
+	(zone
+		(net 1)
+		(net_name "GND")
+		(layer "In1.Cu")
+		(hatch edge 0.5)
 		(priority 1)
 		(connect_pads yes
@@
 			)
 		)
+	)
+	(zone
+		(net 1)
+		(net_name "GND")
+		(layer "In2.Cu")
+		(hatch edge 0.5)
+		(priority 1)
+		(connect_pads yes
+			(clearance 0.5)
+		)
+		(min_thickness 0.25)
+		(filled_areas_thickness no)
+		(fill yes
+			(thermal_gap 0.5)
+			(thermal_bridge_width 0.5)
+		)
+		(polygon
+			(pts
+				(xy 123.39 98.8) (xy 123.39 120.71) (xy 168.3 120.71) (xy 168.3 98.8)
+			)
+		)

Commit message: New Fuse+Gerbers
Parts:
- F1: value MF-RHS800-0 -> SF-1206HHA800R-2; footprint MF-RHS800-0:MFRHS8000 -> SF-1206HHA800R-2:SF1206HHA800R2
- moved F1 0.95 mm to (151.8, 103.5)
Changed lines of the file:
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@@
 		(embedded_fonts no)
 	)
-	(footprint "MF-RHS800-0:MFRHS8000"
+	(footprint "SF-1206HHA800R-2:SF1206HHA800R2"
 		(layer "F.Cu")
-		(at 151.8275 102.5925 -90)
-		(descr "MF-RHS800-0-2")
-		(tags "Resettable Fuse")
+		(at 151.8275 103.54 -90)
+		(descr "SF-1206HHA800R-2")
+		(tags "Fuse")
 		(property "Reference" "F1"
-			(at 0.5175 2.9875 0)
+			(at -1.4825 3.0475 180)
 			(layer "F.SilkS")
 			(effects
@@
 			)
 		)
-		(property "Value" "MF-RHS800-0"
-			(at 2.55 0 90)
+		(property "Value" "SF-1206HHA800R-2"
+			(at 0 0 90)
 			(layer "F.SilkS")
 			(hide yes)
@@
 			)
 		)
-		(property "Datasheet" "https://www.bourns.com/docs/Product-Datasheets/MF-RHS.pdf"
+		(property "Datasheet" "https://www.bourns.com/docs/Product-Datasheets/SF-1206HHA-R.pdf"
 			(at 0 0 90)
 			(layer "F.Fab")
@@
 			)
 		)
-		(property "Description" "PTC 8.0A 16V RADIAL LEADED HI-TEMP"
+		(property "Description" "1206 high-current met-foil. 8A Auto"
 			(at 0 0 90)
 			(layer "F.Fab")
@@
 			)
 		)
-		(property "Height" "24.7"
-			(at 0 0 270)
-			(unlocked yes)
-			(layer "F.Fab")
-			(hide yes)
-			(effects
-				(font
-					(size 1 1)
-					(thickness 0.15)
-				)
-			)
-		)
-		(property "Mouser Part Number" "652-MF-RHS800-0"
-			(at 0 0 270)
-			(unlocked yes)
-			(layer "F.Fab")
-			(hide yes)
-			(effects
-				(font
-					(size 1 1)
-					(thickness 0.15)
-				)
-			)
-		)
-		(property "Mouser Price/Stock" "https://www.mouser.co.uk/ProductDetail/Bourns/MF-RHS800-0?qs=mELouGlnn3db4Obe02aVdw%3D%3D"
+		(property "Height" "1.2"
+			(at 0 0 270)
+			(unlocked yes)
+			(layer "F.Fab")
+			(hide yes)
+			(effects
+				(font
+					(size 1 1)
+					(thickness 0.15)
+				)
+			)
+		)
+		(property "Mouser Part Number" "652-SF-1206HHA800R-2"
+			(at 0 0 270)
+			(unlocked yes)
+			(layer "F.Fab")
+			(hide yes)
+			(effects
+				(font
+					(size 1 1)
+					(thickness 0.15)
+				)
+			)
+		)
+		(property "Mouser Price/Stock" "https://www.mouser.co.uk/ProductDetail/Bourns/SF-1206HHA800R-2?qs=Imq1NPwxi77tr2%2FYGnM5Ig%3D%3D"
 			(at 0 0 270)
 			(unlocked yes)
@@
 			)
 		)
-		(property "Manufacturer_Part_Number" "MF-RHS800-0"
+		(property "Manufacturer_Part_Number" "SF-1206HHA800R-2"
 			(at 0 0 270)
 			(unlocked yes)
@@
 		(sheetname "/")
 		(sheetfile "BIFROST-3S.kicad_sch")
-		(attr through_hole)
-		(fp_line
-			(start -3.85 1.8)
-			(end 8.95 1.8)
+		(attr smd)
+		(fp_line
+			(start -0.8 0.825)
+			(end 0.8 0.825)
 			(stroke
 				(width 0.2)
@@
 		)
 		(fp_line
-			(start 8.95 1.8)
-			(end 8.95 -1.8)
+			(start -3 0)
+			(end -3 0)
+			(stroke
+				(width 0.1)
+				(type solid)
+			)
+			(layer "F.SilkS")
+		)
+		(fp_line
+			(start -2.9 0)
+			(end -2.9 0)
+			(stroke
+				(width 0.1)
+				(type solid)
+			)
+			(layer "F.SilkS")
+		)
+		(fp_line
+			(start -0.8 -0.825)
+			(end 0.8 -0.825)
 			(stroke
 				(width 0.2)
@@
 			(layer "F.SilkS")
 		)
-		(fp_line
-			(start -4.45 0)
-			(end -4.45 0)
-			(stroke
-				(width 0.1)
-				(type solid)
-			)
-			(layer "F.SilkS")
-		)
-		(fp_line
-			(start -4.35 0)
-			(end -4.35 0)
-			(stroke
-				(width 0.1)
-				(type solid)
-			)
-			(layer "F.SilkS")
-		)
-		(fp_line
-			(start -3.85 -1.8)
-			(end -3.85 1.8)
-			(stroke
-				(width 0.2)
-				(type solid)
-			)
-			(layer "F.SilkS")
-		)
-		(fp_line
-			(start 8.95 -1.8)
-			(end -3.85 -1.8)
-			(stroke
-				(width 0.2)
-				(type solid)
-			)
-			(layer "F.SilkS")
-		)
 		(fp_arc
-			(start -4.45 0)
-			(mid -4.4 -0.05)
-			(end -4.35 0)
+			(start -3 0)
+			(mid -2.95 -0.05)
+			(end -2.9 0)
 			(stroke
 				(width 0.1)
@@
 		)
 		(fp_arc
-			(start -4.35 0)
-			(mid -4.4 0.05)
-			(end -4.45 0)
-			(stroke
-				(width 0.1)
-				(type solid)
-			)
-			(layer "F.SilkS")
-		)
-		(fp_line
-			(start -4.15 2.15)
-			(end -4.15 -2.075)
-			(stroke
-				(width 0.1)
-				(type solid)
-			)
-			(layer "F.CrtYd")
-		)
-		(fp_line
-			(start 9.225 2.15)
-			(end -4.15 2.15)
-			(stroke
-				(width 0.1)
-				(type solid)
-			)
-			(layer "F.CrtYd")
-		)
-		(fp_line
-			(start -4.15 -2.075)
-			(end 9.225 -2.075)
-			(stroke
-				(width 0.1)
-				(type solid)
-			)
-			(layer "F.CrtYd")
-		)
-		(fp_line
-			(start 9.225 -2.075)
-			(end 9.225 2.15)
-			(stroke
-				(width 0.1)
-				(type solid)
-			)
-			(layer "F.CrtYd")
-		)
-		(fp_line
-			(start -3.85 1.8)
-			(end 8.95 1.8)
-			(stroke
-				(width 0.1)
-				(type solid)
-			)
-			(layer "F.Fab")
-		)
-		(fp_line
-			(start 8.95 1.8)
-			(end 8.95 -1.8)
-			(stroke
-				(width 0.1)
-				(type solid)
-			)
-			(layer "F.Fab")
-		)
-		(fp_line
-			(start -3.85 -1.8)
-			(end -3.85 1.8)
-			(stroke
-				(width 0.1)
-				(type solid)
-			)
-			(layer "F.Fab")
-		)
-		(fp_line
-			(start 8.95 -1.8)
-			(end -3.85 -1.8)
+			(start -2.9 0)
+			(mid -2.95 0.05)
+			(end -3 0)
+			(stroke
+				(width 0.1)
+				(type solid)
+			)
+			(layer "F.SilkS")
+		)
+		(fp_line
+			(start -3.35 1.825)
+			(end -3.35 -1.825)
+			(stroke
+				(width 0.1)
+				(type solid)
+			)
+			(layer "F.CrtYd")
+		)
+		(fp_line
+			(start 3.35 1.825)
+			(end -3.35 1.825)
+			(stroke
+				(width 0.1)
+				(type solid)
+			)
+			(layer "F.CrtYd")
+		)
+		(fp_line
+			(start -3.35 -1.825)
+			(end 3.35 -1.825)
+			(stroke
+				(width 0.1)
+				(type solid)
+			)
+			(layer "F.CrtYd")
+		)
+		(fp_line
+			(start 3.35 -1.825)
+			(end 3.35 1.825)
+			(stroke
+				(width 0.1)
+				(type solid)
+			)
+			(layer "F.CrtYd")
+		)
+		(fp_line
+			(start -1.6 0.825)
+			(end 1.6 0.825)
+			(stroke
+				(width 0.1)
+				(type solid)
+			)
+			(layer "F.Fab")
+		)
+		(fp_line
+			(start 1.6 0.825)
+			(end 1.6 -0.825)
+			(stroke
+				(width 0.1)
+				(type solid)
+			)
+			(layer "F.Fab")
+		)
+		(fp_line
+			(start -1.6 -0.825)
+			(end -1.6 0.825)
+			(stroke
+				(width 0.1)
+				(type solid)
+			)
+			(layer "F.Fab")
+		)
+		(fp_line
+			(start 1.6 -0.825)
+			(end -1.6 -0.825)
 			(stroke
 				(width 0.1)
@@
 		)
 		(fp_text user "${REFERENCE}"
-			(at 0.5175 2.9875 0)
+			(at -1.4825 3.0475 180)
 			(layer "F.Fab")
 			(effects
@@
 			)
 		)
-		(pad "1" thru_hole rect
-			(at 0 0 270)
-			(size 1.8 1.8)
-			(drill 1.2)
-			(layers "*.Cu" "*.Mask")
-			(remove_unused_layers no)
+		(pad "1" smd rect
+			(at -1.725 0 270)
+			(size 1.25 1.65)
+			(layers "F.Cu" "F.Mask" "F.Paste")
 			(net 6 "/PACK+_RAW")
 			(pinfunction "1")
 			(pintype "passive")
 		)
-		(pad "2" thru_hole circle
-			(at 5.1 0 270)
-			(size 1.8 1.8)
-			(drill 1.2)
-			(layers "*.Cu" "*.Mask")
-			(remove_unused_layers no)
+		(pad "2" smd rect
+			(at 1.725 0 270)
+			(size 1.25 1.65)
+			(layers "F.Cu" "F.Mask" "F.Paste")
 			(net 3 "/+BATT")
 			(pinfunction "2")
@@
 		)
 		(embedded_fonts no)
-		(model "${KIPRJMOD}/CERBERUS-3S FOOTPRINTS/LIB_MF-RHS800-0/MF-RHS800-0/3D/MF-RHS800-0.stp"
+		(model "${KIPRJMOD}/CERBERUS-3S FOOTPRINTS/LIB_SF-1206HHA800R-2/SF-1206HHA800R-2/3D/SF-1206HHA800R-2.stp"
 			(offset
-				(xyz 0 0 0)
+				(xyz 0.05999999776 0.8199999805 0.04999999999)
 			)
 			(scale
@@
 			)
 			(rotate
-				(xyz 0 0 0)
-			)
-		)
+				(xyz -90 0 0)
+			)
+		)
