File: BIFROST-3S.kicad_sch (KiCad schematic)
At the start: 6 parts, among them J1 B6B-XH-A_LF__SN_, J2 Conn_01x12, J3 B4B-XH-A_LF__SN_, J4 XT30PW-M

Commit message: Fixed Vias+Pins
Connections:
- net BQ2_TS1: now also J2.7 (Pin_7), J3.1; no longer J2.10 (Pin_10), J3.4
- net BQ2_TS2: now also J2.8 (Pin_8), J3.2; no longer J2.9 (Pin_9), J3.3
- net BQ2_TS3: now also J2.9 (Pin_9), J3.3; no longer J2.8 (Pin_8), J3.2
- net GND: now also J2.10 (Pin_10), J3.4; no longer J2.7 (Pin_7), J3.1
Changed lines of the file:
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@@
+	(wire
+		(pts
+			(xy 39.37 54.61) (xy 34.29 54.61)
+		)
+		(stroke
+			(width 0)
+			(type default)
+		)
+	)
 	(wire
 		(pts
@@
 	(wire
 		(pts
-			(xy 39.37 46.99) (xy 27.94 46.99)
-		)
-		(stroke
-			(width 0)
-			(type default)
-		)
-	)
-	(wire
-		(pts
 			(xy 160.02 29.21) (xy 163.83 29.21)
 		)
@@
 	(wire
 		(pts
-			(xy 175.26 53.34) (xy 175.26 63.5)
+			(xy 34.29 54.61) (xy 34.29 55.88)
 		)
 		(stroke
@@
 	(wire
 		(pts
+			(xy 182.88 53.34) (xy 182.88 63.5)
+		)
+		(stroke
+			(width 0)
+			(type default)
+		)
+	)
+	(wire
+		(pts
 			(xy 22.86 35.56) (xy 22.86 38.1)
 		)
@@
 		(pts
 			(xy 130.81 26.67) (xy 125.73 26.67)
-		)
-		(stroke
-			(width 0)
-			(type default)
-		)
-	)
-	(wire
-		(pts
-			(xy 27.94 46.99) (xy 27.94 53.34)
 		)
 		(stroke
@@
 	)
 	(label "BQ2_TS1"
-		(at 39.37 54.61 180)
+		(at 39.37 46.99 180)
 		(effects
 			(font
@@
 	)
 	(label "BQ2_TS2"
-		(at 180.34 53.34 270)
+		(at 177.8 53.34 270)
 		(effects
 			(font
@@
 	)
 	(label "BQ2_TS3"
-		(at 39.37 49.53 180)
+		(at 39.37 52.07 180)
 		(effects
 			(font
@@
 	)
 	(label "BQ2_TS3"
-		(at 177.8 53.34 270)
+		(at 180.34 53.34 270)
 		(effects
 			(font
@@
 	)
 	(label "BQ2_TS1"
-		(at 182.88 53.34 270)
+		(at 175.26 53.34 270)
 		(effects
 			(font
@@
 	)
 	(label "BQ2_TS2"
-		(at 39.37 52.07 180)
+		(at 39.37 49.53 180)
 		(effects
 			(font
@@
 		(on_board yes)
 		(dnp no)
-		(fields_autoplaced yes)
 		(property "Reference" "#PWR08"
 			(at 185.42 69.85 0)
@@
 		)
 		(property "Value" "GND"
-			(at 185.42 68.58 0)
+			(at 180.594 68.834 0)
 			(effects
 				(font
@@
 	(symbol
 		(lib_id "power:GND")
-		(at 27.94 53.34 0)
+		(at 34.29 55.88 0)
 		(unit 1)
 		(exclude_from_sim no)
@@
 		(fields_autoplaced yes)
 		(property "Reference" "#PWR05"
-			(at 27.94 59.69 0)
+			(at 34.29 62.23 0)
 			(effects
 				(font
@@
 		)
 		(property "Value" "GND"
-			(at 27.94 58.42 0)
+			(at 34.29 60.96 0)
 			(effects
 				(font
@@
 		)
 		(property "Footprint" ""
-			(at 27.94 53.34 0)
+			(at 34.29 55.88 0)
 			(effects
 				(font
@@
 		)
 		(property "Datasheet" ""
-			(at 27.94 53.34 0)
+			(at 34.29 55.88 0)
 			(effects
 				(font
@@
 		)
 		(property "Description" "Power symbol creates a global label with name \"GND\" , ground"
-			(at 27.94 53.34 0)
+			(at 34.29 55.88 0)
 			(effects
 				(font
@@
 	(symbol
 		(lib_id "power:GND")
-		(at 175.26 63.5 0)
+		(at 182.88 63.5 0)
 		(unit 1)
 		(exclude_from_sim no)
@@
 		(dnp no)
 		(property "Reference" "#PWR07"
-			(at 175.26 69.85 0)
+			(at 182.88 69.85 0)
 			(effects
 				(font
@@
 		)
 		(property "Value" "GND"
-			(at 177.546 68.834 0)
+			(at 187.96 68.834 0)
 			(effects
 				(font
@@
 		)
 		(property "Footprint" ""
-			(at 175.26 63.5 0)
+			(at 182.88 63.5 0)
 			(effects
 				(font
@@
 		)
 		(property "Datasheet" ""
-			(at 175.26 63.5 0)
+			(at 182.88 63.5 0)
 			(effects
 				(font
@@
 		)
 		(property "Description" "Power symbol creates a global label with name \"GND\" , ground"
-			(at 175.26 63.5 0)
-			(effects
-				(font
+			(at 182.88 63.5 0)
+			(effects
+				(font
